Commit message: Added MIT license header in all files and added make_unique C++14 in Pointers.h

File: doc/models/robot.urdf (robot description, URDF)
Before this commit: robot gpa546, 4 links, 3 joints
Joints:
- joint joint_piece1: origin xyz=0 0 0.4 rpy=-1.57079632679 0 0 -> xyz=0 0 0.4 rpy=0 0 0

Commit message: Removed joint_state_publisher and robot_state_publisher from roslaunch file

File: doc/models/robot.urdf (robot description, URDF)
Before this commit: robot gpa546, 4 links, 3 joints
Joints:
- joint joint_piece1: origin xyz=0 0 0.4 rpy=0 0 0 -> xyz=0 0 0.4 rpy=-1.57079632679 0 0

Commit message: Fixed URDF model. Added more verbosity in RobotStatePublisher for logging purpose

File: doc/models/robot.urdf (robot description, URDF)
Before this commit: robot gpa546, 4 links, 3 joints
Joints:
- joint joint_piece1: origin xyz=0 0 0.4 rpy=-1.57079632679 0 0 -> xyz=0 0 1 rpy=1.57079632679 0 0
- joint joint_piece2: origin xyz=0 -2 0 rpy=0 0 0 -> xyz=0 2 0 rpy=0 0 0
